Commit message: 20211205

File: urdf/single_joint_actuator.urdf.xacro (robot description, xacro)
@@ -40,5 +40,5 @@
     </visual>
    </link>
-   <joint name="joint1" type="continuous">
+   <joint name="my_joint" type="continuous">
      <axis xyz="0 0 1"/>
      <origin rpy="0 0 0" xyz="0.02 0 0.01"/>
